File: locator_beacon.kicad_pcb (KiCad board)
At the start: 2 copper layers, 50.9 x 20.8 mm, 35 parts, among them J1 Conn_01x02, J2 Conn_01x02, Q1 DMN6140, Q2 DMN6140, Q3 DMN6140, Q4 DMN6140, U1 MC34063AD, U13 Pico, U3 MIC4606

Commit message: Tweaks
Parts:
- removed L2: 10u, Inductor_SMD:L_1210_3225Metric
- added C3: 220n, Capacitor_SMD:C_0603_1608Metric, F.Cu at (162.3, 77.5)
- C15, C17: value 10u -> 1.5n
- C5: value 10u -> 220n
- D3: value B120-E3 -> DSS16U
- L1: footprint Inductor_SMD:L_1210_3225Metric -> Inductor_SMD:L_Taiyo-Yuden_MD-4040
- moved REF** 1.45 mm to (157.5, 83.6)
- moved C5 0.52 mm to (162.3, 79.0)
- moved R1 0.26 mm to (157.1, 78.7)
- moved C17 0.25 mm to (153.8, 78.7)
- moved TP6 0.18 mm to (143.6, 73.5)
- moved C4 0.13 mm to (149.2, 74.0)
Connections:
- C5 pad 2: Net-(C5-Pad2) -> GND
- U13 pad 29: unconnected-(U13-GPIO22-Pad29) -> /amplifier/EN
- U3 pad 2: Vdrive -> /amplifier/EN
Routing:
- net /amplifier/EN: track 0.00 -> 10.1 mm
- net Vdrive: track 37.3 -> 31.5 mm
- net GND: track 60.3 -> 63.2 mm
- net /amplifier/OUT_B: track 36.5 -> 39.4 mm
- net Net-(C5-Pad2): track 2.72 -> 0.00 mm
