File: locator_beacon.kicad_sch (KiCad schematic)
At the start: 2 parts, among them J1 Conn_01x02, U13 Pico

Commit message: Tweaks
Parts:
- J1: now left out of the parts list
Connections:
- net amplifier/EN: now reaches U13.29 (GPIO22)
Other:
- sheet amplifier ports: added EN; removed none
Changed lines of the file:
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@@
+    (stroke (width 0) (type default))
+  )
+  (wire (pts (xy 130.81 109.22) (xy 130.81 137.16))
     (stroke (width 0) (type default))
   )
@@
     (stroke (width 0) (type default))
   )
+  (wire (pts (xy 115.57 109.22) (xy 130.81 109.22))
+    (stroke (width 0) (type default))
+  )
   (wire (pts (xy 123.19 83.82) (xy 115.57 83.82))
     (stroke (width 0) (type default))
@@
     (stroke (width 0) (type default))
   )
+  (wire (pts (xy 68.58 116.84) (xy 66.04 116.84))
+    (stroke (width 0) (type default))
+  )
   (wire (pts (xy 115.57 111.76) (xy 123.19 111.76))
     (stroke (width 0) (type default))
   )
+  (wire (pts (xy 130.81 137.16) (xy 68.58 137.16))
+    (stroke (width 0) (type default))
+  )
   (wire (pts (xy 115.57 99.06) (xy 123.19 99.06))
     (stroke (width 0) (type default))
@@
     (stroke (width 0) (type default))
   )
+  (wire (pts (xy 68.58 137.16) (xy 68.58 116.84))
+    (stroke (width 0) (type default))
+  )
   (wire (pts (xy 115.57 124.46) (xy 123.19 124.46))
     (stroke (width 0) (type default))
@@
   )
   (symbol (lib_id "Connector_Generic:Conn_01x02") (at 27.94 119.38 0) (mirror y) (unit 1)
-    (in_bom yes) (on_board yes) (dnp no)
+    (in_bom no) (on_board yes) (dnp no)
     (property "Reference" "J1" (at 25.4 119.38 0)
       (effects (font (size 1.27 1.27)) (justify left))
@@
     )
     (property "Datasheet" "~" (at 27.94 119.38 0)
+      (effects (font (size 1.27 1.27)) hide)
+    )
+    (property "Sim.Enable" "0" (at 27.94 119.38 0)
       (effects (font (size 1.27 1.27)) hide)
     )
@@
     )
   )
-  (sheet (at 49.53 118.11) (size 16.51 5.08) (fields_autoplaced)
+  (sheet (at 49.53 115.57) (size 16.51 7.62) (fields_autoplaced)
     (stroke (width 0.1524) (type solid))
     (fill (color 0 0 0 0.0000))
-    (property "Sheetname" "amplifier" (at 49.53 117.3984 0)
+    (property "Sheetname" "amplifier" (at 49.53 114.8584 0)
       (effects (font (size 1.27 1.27)) (justify left bottom))
     )
@@
       (effects (font (size 1.27 1.27)) (justify right))
     )
+    (pin "EN" input (at 66.04 116.84 0)
+      (effects (font (size 1.27 1.27)) (justify right))
+    )
