File: locator_beacon.kicad_sch (KiCad schematic)
At the start: 2 parts, among them J1 Conn_01x02, U13 Pico

Commit message: changes
Parts:
- added D1: DSS16U, Diode_SMD:D_SOD-123, symbol Diode:B120-E3
- added J3, J6: Conn_01x01, Connector_PinHeader_2.54mm:PinHeader_1x01_P2.54mm_Vertical, symbol Connector_Generic:Conn_01x01
- added J4: OSHW logo, Symbol:OSHW-Logo_5.7x6mm_Copper, symbol Connector_Generic:Conn_01x01
- added J7: Conn_01x02, Connector_PinHeader_2.54mm:PinHeader_1x02_P2.54mm_Vertical, symbol Connector_Generic:Conn_01x02
- J1: footprint Connector_PinHeader_2.54mm:PinHeader_1x02_P2.54mm_Horizontal -> custom:SAMTEC_TSM-102-01-L-SH; symbol Connector_Generic:Conn_01x02 -> custom_symbols:TSM-102-01-L-SH; MANUFACTURER (none) -> Samtec; PARTREV (none) -> R; STANDARD (none) -> Manufacturer Recommendations; now in the parts list
- U13: footprint custom:rp_pico -> custom:RPi_pico
Connections:
- net +BATT: now also D1.2 (A); no longer U13.39 (VSYS)
- net amplifier/EN: now also U13.25 (GPIO19), J3.1 (Pin_1); no longer U13.29 (GPIO22)
- net amplifier/OUT_A: now also J1.02; no longer J1.2 (Pin_2)
- net amplifier/OUT_B: now also J1.01; no longer J1.1 (Pin_1)
- net amplifier/SIG_IN: now also J7.1 (Pin_1)
- net amplifier/~{SIG_IN}: now also J7.2 (Pin_2)
- net power/EN: now reaches U13.2 (GPIO1)
- net power/EN: now also J6.1 (Pin_1)
- new net: D1.1 (K), U13.39 (VSYS)
Other:
- sheet power ports: added EN; removed none
- moved on the sheet: J1
Changed lines of the file:
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@@
   (junction (at 123.19 124.46) (diameter 0) (color 0 0 0 0)
   )
+  (junction (at 73.66 121.92) (diameter 0) (color 0 0 0 0)
+  )
+  (junction (at 68.58 116.84) (diameter 0) (color 0 0 0 0)
+  )
   (junction (at 74.93 124.46) (diameter 0) (color 0 0 0 0)
   )
   (junction (at 74.93 99.06) (diameter 0) (color 0 0 0 0)
   )
+  (junction (at 73.66 119.38) (diameter 0) (color 0 0 0 0)
+  )
   (junction (at 74.93 111.76) (diameter 0) (color 0 0 0 0)
   )
@@
   (junction (at 123.19 99.06) (diameter 0) (color 0 0 0 0)
   )
+  (junction (at 74.93 83.82) (diameter 0) (color 0 0 0 0)
+  )
+  (wire (pts (xy 73.66 121.92) (xy 80.01 121.92))
+    (stroke (width 0) (type default))
+  )
   (wire (pts (xy 123.19 124.46) (xy 123.19 111.76))
     (stroke (width 0) (type default))
   )
+  (wire (pts (xy 115.57 119.38) (xy 132.08 119.38))
+    (stroke (width 0) (type default))
+  )
+  (wire (pts (xy 80.01 83.82) (xy 74.93 83.82))
+    (stroke (width 0) (type default))
+  )
   (wire (pts (xy 74.93 111.76) (xy 80.01 111.76))
     (stroke (width 0) (type default))
   )
-  (wire (pts (xy 66.04 119.38) (xy 80.01 119.38))
+  (wire (pts (xy 66.04 121.92) (xy 73.66 121.92))
     (stroke (width 0) (type default))
   )
@@
     (stroke (width 0) (type default))
   )
+  (wire (pts (xy 66.04 119.38) (xy 73.66 119.38))
+    (stroke (width 0) (type default))
+  )
+  (wire (pts (xy 74.93 48.26) (xy 107.95 48.26))
+    (stroke (width 0) (type default))
+  )
   (wire (pts (xy 74.93 86.36) (xy 80.01 86.36))
     (stroke (width 0) (type default))
   )
-  (wire (pts (xy 130.81 109.22) (xy 130.81 137.16))
-    (stroke (width 0) (type default))
-  )
   (wire (pts (xy 123.19 80.01) (xy 123.19 83.82))
     (stroke (width 0) (type default))
@@
     (stroke (width 0) (type default))
   )
+  (wire (pts (xy 74.93 83.82) (xy 74.93 48.26))
+    (stroke (width 0) (type default))
+  )
   (wire (pts (xy 33.02 121.92) (xy 49.53 121.92))
     (stroke (width 0) (type default))
@@
     (stroke (width 0) (type default))
   )
-  (wire (pts (xy 115.57 109.22) (xy 130.81 109.22))
-    (stroke (width 0) (type default))
-  )
-  (wire (pts (xy 123.19 83.82) (xy 115.57 83.82))
-    (stroke (width 0) (type default))
-  )
   (wire (pts (xy 74.93 124.46) (xy 80.01 124.46))
     (stroke (width 0) (type default))
   )
+  (wire (pts (xy 132.08 119.38) (xy 132.08 137.16))
+    (stroke (width 0) (type default))
+  )
   (wire (pts (xy 74.93 138.43) (xy 74.93 124.46))
     (stroke (width 0) (type default))
@@
     (stroke (width 0) (type default))
   )
+  (wire (pts (xy 73.66 119.38) (xy 80.01 119.38))
+    (stroke (width 0) (type default))
+  )
   (wire (pts (xy 123.19 99.06) (xy 123.19 86.36))
     (stroke (width 0) (type default))
@@
     (stroke (width 0) (type default))
   )
-  (wire (pts (xy 130.81 137.16) (xy 68.58 137.16))
+  (wire (pts (xy 132.08 137.16) (xy 68.58 137.16))
     (stroke (width 0) (type default))
   )
@@
     (stroke (width 0) (type default))
   )
-  (wire (pts (xy 66.04 121.92) (xy 80.01 121.92))
-    (stroke (width 0) (type default))
-  )
-  (symbol (lib_id "Connector_Generic:Conn_01x02") (at 27.94 119.38 0) (mirror y) (unit 1)
-    (in_bom no) (on_board yes) (dnp no)
-    (property "Reference" "J1" (at 25.4 119.38 0)
+  (symbol (lib_id "Connector_Generic:Conn_01x02") (at 68.58 121.92 180) (unit 1)
+    (in_bom yes) (on_board yes) (dnp yes) (fields_autoplaced)
+    (property "Reference" "J7" (at 68.58 113.03 0)
+      (effects (font (size 1.27 1.27)))
+    )
+    (property "Value" "Conn_01x02" (at 68.58 115.57 0)
+      (effects (font (size 1.27 1.27)))
+    )
+    (property "Footprint" "Connector_PinHeader_2.54mm:PinHeader_1x02_P2.54mm_Vertical" (at 68.58 121.92 0)
+      (effects (font (size 1.27 1.27)) hide)
+    )
+    (property "Datasheet" "~" (at 68.58 121.92 0)
+      (effects (font (size 1.27 1.27)) hide)
+    )
+    (pin "1")
+    (pin "2")
+    (instances
+      (project "locator_beacon"
+        (path "/2e37f9ca-1f81-48a3-bbbb-9eab5c177622"
+          (reference "J7") (unit 1)
+        )
+      )
+    )
+  )
+  (symbol (lib_id "custom_symbols:TSM-102-01-L-SH") (at 20.32 121.92 0) (mirror y) (unit 1)
+    (in_bom yes) (on_board yes) (dnp no)
+    (property "Reference" "J1" (at 17.78 121.92 0)
       (effects (font (size 1.27 1.27)) (justify left))
     )
-    (property "Value" "Conn_01x02" (at 25.4 121.92 0)
+    (property "Value" "Conn_01x02" (at 17.78 124.46 0)
       (effects (font (size 1.27 1.27)) (justify left))
     )
-    (property "Footprint" "Connector_PinHeader_2.54mm:PinHeader_1x02_P2.54mm_Horizontal" (at 27.94 119.38 0)
-      (effects (font (size 1.27 1.27)) hide)
-    )
-    (property "Datasheet" "~" (at 27.94 119.38 0)
-      (effects (font (size 1.27 1.27)) hide)
-    )
-    (property "Sim.Enable" "0" (at 27.94 119.38 0)
+    (property "Footprint" "custom:SAMTEC_TSM-102-01-L-SH" (at 17.78 111.76 0)
+      (effects (font (size 1.27 1.27)) (justify bottom) hide)
+    )
+    (property "Datasheet" "~" (at 20.32 121.92 0)
+      (effects (font (size 1.27 1.27)) hide)
+    )
+    (property "Sim.Enable" "0" (at 20.32 121.92 0)
+      (effects (font (size 1.27 1.27)) hide)
+    )
+    (property "PARTREV" "R" (at 20.32 121.92 0)
+      (effects (font (size 1.27 1.27)) (justify bottom) hide)
+    )
+    (property "STANDARD" "Manufacturer Recommendations" (at 19.05 114.3 0)
+      (effects (font (size 1.27 1.27)) (justify bottom) hide)
+    )
+    (property "MANUFACTURER" "Samtec" (at 20.32 121.92 0)
+      (effects (font (size 1.27 1.27)) (justify bottom) hide)
+    )
+    (pin "02")
+    (pin "01")
+    (instances
+      (project "locator_beacon"
+        (path "/2e37f9ca-1f81-48a3-bbbb-9eab5c177622"
+          (reference "J1") (unit 1)
+        )
+      )
+    )
+  )
+  (symbol (lib_id "Diode:B120-E3") (at 119.38 83.82 0) (unit 1)
+    (in_bom yes) (on_board yes) (dnp no) (fields_autoplaced)
+    (property "Reference" "D1" (at 119.0625 77.47 0)
+      (effects (font (size 1.27 1.27)))
+    )
+    (property "Value" "DSS16U" (at 119.0625 80.01 0)
+      (effects (font (size 1.27 1.27)))
+    )
+    (property "Footprint" "Diode_SMD:D_SOD-123" (at 119.38 88.265 0)
+      (effects (font (size 1.27 1.27)) hide)
+    )
+    (property "Datasheet" "http://www.vishay.com/docs/88946/b120.pdf" (at 119.38 83.82 0)
       (effects (font (size 1.27 1.27)) hide)
     )
@@
       (project "locator_beacon"
         (path "/2e37f9ca-1f81-48a3-bbbb-9eab5c177622"
-          (reference "J1") (unit 1)
+          (reference "D1") (unit 1)
         )
       )
@@
       (effects (font (size 1.27 1.27)))
     )
-    (property "Footprint" "custom:rp_pico" (at 97.79 105.41 90)
+    (property "Footprint" "custom:RPi_pico" (at 97.79 105.41 90)
       (effects (font (size 1.27 1.27)) hide)
     )
@@
     )
   )
+  (symbol (lib_id "Connector_Generic:Conn_01x01") (at 39.37 152.4 0) (unit 1)
+    (in_bom yes) (on_board yes) (dnp no) (fields_autoplaced)
+    (property "Reference" "J4" (at 41.91 151.13 0)
+      (effects (font (size 1.27 1.27)) (justify left) hide)
+    )
+    (property "Value" "OSHW logo" (at 41.91 153.67 0)
+      (effects (font (size 1.27 1.27)) (justify left))
+    )
+    (property "Footprint" "Symbol:OSHW-Logo_5.7x6mm_Copper" (at 39.37 152.4 0)
+      (effects (font (size 1.27 1.27)) hide)
+    )
+    (property "Datasheet" "~" (at 39.37 152.4 0)
+      (effects (font (size 1.27 1.27)) hide)
+    )
+    (pin "1")
+    (instances
+      (project "locator_beacon"
+        (path "/2e37f9ca-1f81-48a3-bbbb-9eab5c177622"
+          (reference "J4") (unit 1)
+        )
+      )
+    )
+  )
   (symbol (lib_id "power:GND") (at 123.19 138.43 0) (unit 1)
     (in_bom yes) (on_board yes) (dnp no) (fields_autoplaced)
@@
         (path "/2e37f9ca-1f81-48a3-bbbb-9eab5c177622"
           (reference "#PWR020") (unit 1)
+        )
+      )
+    )
+  )
+  (symbol (lib_id "Connector_Generic:Conn_01x01") (at 69.85 83.82 180) (unit 1)
+    (in_bom yes) (on_board yes) (dnp no) (fields_autoplaced)
+    (property "Reference" "J6" (at 69.85 77.47 0)
+      (effects (font (size 1.27 1.27)))
+    )
+    (property "Value" "Conn_01x01" (at 69.85 80.01 0)
+      (effects (font (size 1.27 1.27)))
+    )
+    (property "Footprint" "Connector_PinHeader_2.54mm:PinHeader_1x01_P2.54mm_Vertical" (at 69.85 83.82 0)
+      (effects (font (size 1.27 1.27)) hide)
+    )
+    (property "Datasheet" "~" (at 69.85 83.82 0)
+      (effects (font (size 1.27 1.27)) hide)
+    )
+    (pin "1")
+    (instances
+      (project "locator_beacon"
+        (path "/2e37f9ca-1f81-48a3-bbbb-9eab5c177622"
+          (reference "J6") (unit 1)
+        )
+      )
+    )
+  )
+  (symbol (lib_id "Connector_Generic:Conn_01x01") (at 68.58 111.76 90) (unit 1)
+    (in_bom yes) (on_board yes) (dnp yes) (fields_autoplaced)
+    (property "Reference" "J3" (at 71.12 110.49 90)
+      (effects (font (size 1.27 1.27)) (justify right))
+    )
+    (property "Value" "Conn_01x01" (at 71.12 113.03 90)
+      (effects (font (size 1.27 1.27)) (justify right))
+    )
+    (property "Footprint" "Connector_PinHeader_2.54mm:PinHeader_1x01_P2.54mm_Vertical" (at 68.58 111.76 0)
+      (effects (font (size 1.27 1.27)) hide)
+    )
+    (property "Datasheet" "~" (at 68.58 111.76 0)
+      (effects (font (size 1.27 1.27)) hide)
+    )
+    (pin "1")
+    (instances
+      (project "locator_beacon"
+        (path "/2e37f9ca-1f81-48a3-bbbb-9eab5c177622"
+          (reference "J3") (unit 1)
         )
       )
@@
       (effects (font (size 1.27 1.27)) (justify left top) hide)
     )
-    (instances
+    (pin "EN" input (at 107.95 48.26 180)
+      (effects (font (size 1.27 1.27)) (justify left))
+    )
+    (instances

Commit message: Shrunkified
Parts:
- added J5: Conn_01x02, Connector_PinHeader_2.54mm:PinHeader_1x02_P2.54mm_Vertical, symbol Connector_Generic:Conn_01x02
- J3, J7: now fitted
Connections:
- net GND: now also J5.2 (Pin_2)
- net at D1.1 (K), U13.39 (VSYS): now also J5.1 (Pin_1)
Other:
- moved on the sheet: D1
Changed lines of the file:
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@@
   (junction (at 73.66 121.92) (diameter 0) (color 0 0 0 0)
   )
-  (junction (at 68.58 116.84) (diameter 0) (color 0 0 0 0)
-  )
   (junction (at 74.93 124.46) (diameter 0) (color 0 0 0 0)
   )
   (junction (at 74.93 99.06) (diameter 0) (color 0 0 0 0)
   )
+  (junction (at 123.19 86.36) (diameter 0) (color 0 0 0 0)
+  )
+  (junction (at 132.08 119.38) (diameter 0) (color 0 0 0 0)
+  )
   (junction (at 73.66 119.38) (diameter 0) (color 0 0 0 0)
   )
+  (junction (at 123.19 83.82) (diameter 0) (color 0 0 0 0)
+  )
   (junction (at 74.93 111.76) (diameter 0) (color 0 0 0 0)
   )
@@
     (stroke (width 0) (type default))
   )
-  (wire (pts (xy 123.19 80.01) (xy 123.19 83.82))
-    (stroke (width 0) (type default))
-  )
   (wire (pts (xy 74.93 111.76) (xy 74.93 99.06))
     (stroke (width 0) (type default))
@@
     (stroke (width 0) (type default))
   )
+  (wire (pts (xy 115.57 83.82) (xy 123.19 83.82))
+    (stroke (width 0) (type default))
+  )
   (wire (pts (xy 115.57 99.06) (xy 123.19 99.06))
     (stroke (width 0) (type default))
@@
   )
   (symbol (lib_id "Connector_Generic:Conn_01x02") (at 68.58 121.92 180) (unit 1)
-    (in_bom yes) (on_board yes) (dnp yes) (fields_autoplaced)
+    (in_bom yes) (on_board yes) (dnp no) (fields_autoplaced)
     (property "Reference" "J7" (at 68.58 113.03 0)
       (effects (font (size 1.27 1.27)))
@@
     )
   )
-  (symbol (lib_id "Diode:B120-E3") (at 119.38 83.82 0) (unit 1)
-    (in_bom yes) (on_board yes) (dnp no) (fields_autoplaced)
-    (property "Reference" "D1" (at 119.0625 77.47 0)
-      (effects (font (size 1.27 1.27)))
-    )
-    (property "Value" "DSS16U" (at 119.0625 80.01 0)
-      (effects (font (size 1.27 1.27)))
-    )
-    (property "Footprint" "Diode_SMD:D_SOD-123" (at 119.38 88.265 0)
-      (effects (font (size 1.27 1.27)) hide)
-    )
-    (property "Datasheet" "http://www.vishay.com/docs/88946/b120.pdf" (at 119.38 83.82 0)
+  (symbol (lib_id "Diode:B120-E3") (at 123.19 80.01 90) (unit 1)
+    (in_bom yes) (on_board yes) (dnp no) (fields_autoplaced)
+    (property "Reference" "D1" (at 125.73 79.0575 90)
+      (effects (font (size 1.27 1.27)) (justify right))
+    )
+    (property "Value" "DSS16U" (at 125.73 81.5975 90)
+      (effects (font (size 1.27 1.27)) (justify right))
+    )
+    (property "Footprint" "Diode_SMD:D_SOD-123" (at 127.635 80.01 0)
+      (effects (font (size 1.27 1.27)) hide)
+    )
+    (property "Datasheet" "http://www.vishay.com/docs/88946/b120.pdf" (at 123.19 80.01 0)
       (effects (font (size 1.27 1.27)) hide)
     )
@@
         (path "/2e37f9ca-1f81-48a3-bbbb-9eab5c177622"
           (reference "D1") (unit 1)
+        )
+      )
+    )
+  )
+  (symbol (lib_id "Connector_Generic:Conn_01x02") (at 128.27 83.82 0) (unit 1)
+    (in_bom yes) (on_board yes) (dnp no) (fields_autoplaced)
+    (property "Reference" "J5" (at 130.81 83.82 0)
+      (effects (font (size 1.27 1.27)) (justify left))
+    )
+    (property "Value" "Conn_01x02" (at 130.81 86.36 0)
+      (effects (font (size 1.27 1.27)) (justify left))
+    )
+    (property "Footprint" "Connector_PinHeader_2.54mm:PinHeader_1x02_P2.54mm_Vertical" (at 128.27 83.82 0)
+      (effects (font (size 1.27 1.27)) hide)
+    )
+    (property "Datasheet" "~" (at 128.27 83.82 0)
+      (effects (font (size 1.27 1.27)) hide)
+    )
+    (pin "1")
+    (pin "2")
+    (instances
+      (project "locator_beacon"
+        (path "/2e37f9ca-1f81-48a3-bbbb-9eab5c177622"
+          (reference "J5") (unit 1)
         )
       )
@@
     )
   )
-  (symbol (lib_id "Connector_Generic:Conn_01x01") (at 68.58 111.76 90) (unit 1)
-    (in_bom yes) (on_board yes) (dnp yes) (fields_autoplaced)
-    (property "Reference" "J3" (at 71.12 110.49 90)
+  (symbol (lib_id "Connector_Generic:Conn_01x01") (at 132.08 114.3 90) (unit 1)
+    (in_bom yes) (on_board yes) (dnp no) (fields_autoplaced)
+    (property "Reference" "J3" (at 134.62 113.03 90)
       (effects (font (size 1.27 1.27)) (justify right))
     )
-    (property "Value" "Conn_01x01" (at 71.12 113.03 90)
+    (property "Value" "Conn_01x01" (at 134.62 115.57 90)
       (effects (font (size 1.27 1.27)) (justify right))
     )
-    (property "Footprint" "Connector_PinHeader_2.54mm:PinHeader_1x01_P2.54mm_Vertical" (at 68.58 111.76 0)
-      (effects (font (size 1.27 1.27)) hide)
-    )
-    (property "Datasheet" "~" (at 68.58 111.76 0)
+    (property "Footprint" "Connector_PinHeader_2.54mm:PinHeader_1x01_P2.54mm_Vertical" (at 132.08 114.3 0)
+      (effects (font (size 1.27 1.27)) hide)
+    )
+    (property "Datasheet" "~" (at 132.08 114.3 0)
       (effects (font (size 1.27 1.27)) hide)
     )
@@
     )
   )
-  (symbol (lib_id "power:+BATT") (at 123.19 80.01 0) (unit 1)
-    (in_bom yes) (on_board yes) (dnp no) (fields_autoplaced)
-    (property "Reference" "#PWR01" (at 123.19 83.82 0)
-      (effects (font (size 1.27 1.27)) hide)
-    )
-    (property "Value" "+BATT" (at 123.19 74.93 0)
-      (effects (font (size 1.27 1.27)))
-    )
-    (property "Footprint" "" (at 123.19 80.01 0)
-      (effects (font (size 1.27 1.27)) hide)
-    )
-    (property "Datasheet" "" (at 123.19 80.01 0)
-      (effects (font (size 1.27 1.27)) hide)
-    )
+  (symbol (lib_id "power:+BATT") (at 123.19 76.2 0) (unit 1)
+    (in_bom yes) (on_board yes) (dnp no) (fields_autoplaced)
+    (property "Reference" "#PWR01" (at 123.19 80.01 0)
+      (effects (font (size 1.27 1.27)) hide)
+    )
+    (property "Value" "+BATT" (at 123.19 71.12 0)
+      (effects (font (size 1.27 1.27)))
+    )
+    (property "Footprint" "" (at 123.19 76.2 0)
+      (effects (font (size 1.27 1.27)) hide)
+    )
+    (property "Datasheet" "" (at 123.19 76.2 0)
+      (effects (font (size 1.27 1.27)) hide)
+    )
